File: Drive Board/Drive Board 2018-19.sch (EAGLE design)
At the start: 30 parts, among them IC1 ACS758KCB, IC2 ACS758KCB, IC3 ACS758KCB, IC4 ACS758KCB, K1 JTN-PCB-DC9V

Commit message: Motor drivers added
Parts:
- removed U$7: TRI-BARRIER-TERMINAL, Molex:TRI-BARRIER-TERMINAL
- added C7: 0.33uF, capacitor-wima:C5/5.5
- added C8: 0.1uF, capacitor-wima:C5/5.5
- added IC5: 7812T, adafruit:7812T
- added R8: 330, resistor:R-US_0207/10
- added S1: (no value), switch-dil:DS01E
- added U$1, U$2, U$3, U$4, U$5, U$6: (no value), RSX_Driver_Boards:HPMD18V17
- K1: value JTN-PCB-DC9V -> JTN-PCB-DC6V; device relay:JTN-PCB-DC9V -> relay:JTN-PCB-DC6V
- OK1: value SFH620A -> SFH618A-2; device optocoupler:SFH620A -> optocoupler:SFH618A-2
- R4: value (none) -> 470
- R6, R7: value (none) -> 4.7k
Connections:
- removed net GND: U$7.3, U$7.4
- removed net N$23 (its old number): D1.C, K1G$1.2, R4.2
- removed net N$32: U$7.1, U$7.2
- new net N$29: B2.5V, S1.2
- new net N$31: OK1.A, S1.1
- new net N$34: OK1.C, R8.2
- new net N$35: C7.1, IC5.VI
- new net N$36: C8.1, D1.C, IC5.VO, K1G$1.2, OK1.EMIT, R4.2
- new net N$37: C7.2, C8.2, IC5.GND
- net N$21: now also OK1.COL; no longer OK1.C
Other:
- moved on the sheet: D1, K1, LED1, Q1, R4, R6, R7
