File: Drive Board/Drive Board 2018-19.brd (EAGLE design)
At the start: 379.8 x 115 mm, 113 parts, among them IC1 ACS758KCB, IC2 ACS758KCB, IC3 ACS758KCB, IC4 ACS758KCB, IC5 7812T, IC6 LM741P, K1 G5L, K2 G5L, K3 G5L

Commit message: updated plane thickness
Parts:
- moved LED10 1.27 mm to (143.5, 102.2)
- moved S9 1.27 mm to (139.7, 104.8)
- moved R32 0.63 mm to (135.9, 104.1)
Routing:
- net BATTERY_V+: track 14.2 -> 26.7 mm
- net N$24: track 0.00 -> 3.75 mm
- net ESTOP: track 51.0 -> 54.6 mm
- net OUT4: track 0.00 -> 2.69 mm
- net A5: track 182.0 -> 180.7 mm
- net GND: track 896.3 -> 895.0 mm
Other:
- board size 379.8 x 115 mm -> 379.8 x 116.3 mm
- board text added: "Dylan Lamont 2019"

Commit message: Gerbers added for drive board and arm control pcb
Changed lines of the file:
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@@
 <text x="346.075" y="10.16" size="0.8128" layer="25" rot="R90">OUT B 5</text>
 <text x="350.52" y="10.16" size="0.8128" layer="25" rot="R90">OUT B 4</text>
-<text x="1.27" y="62.865" size="0.5" layer="26" rot="R270">Dylan Lamont 2019</text>
+<text x="1.27" y="62.865" size="0.5" layer="25" rot="R270">Dylan Lamont 2019</text>
 </plain>
 <attributes>
