File: Arm Control Board/ARM Arduino Mega Board.sch (EAGLE design)
At the start: 55 parts, among them X1 5566-2

Commit message: Arm control Board: mirrored arduino, added switches, added mega fit for power, added motor indicator LEDs, added LM7805 for Arduino power regulation
Parts:
- removed B1: ARDUINO_MEGA_R3FULL, SparkFun-Boards:ARDUINO_MEGA_R3FULL
- removed Q13, Q14, Q2, Q3: (no value), adafruit:MOSFET-NREFLOW
- removed R25, R26, R27, R28, R5, R6: 10K, rcl:R-US_R0603
- removed RX: \, wirepad:3,81/1,1
- removed TX: (no value), wirepad:3,81/1,1
- removed X1: 5566-2, con-molex:5566-2
- added ARDUINO_DUE1: (no value), arduino_due_shield:ARDUINO_DUE_SHIELD
- R3, R4: value 10K -> 100K
Connections:
- removed net N$1: Q14.S, R28.1, RX.P
- removed net N$2: Q13.S, R26.1, TX.P
- removed net SCL: B1.21(SCL), Q3.S, R6.1
- removed net SDA: B1.20(SDA), Q2.S, R4.1
- net 12V: now also ARDUINO_DUE1.VIN; no longer B1.VIN, X1-1.S
- net 3.3V: now also ARDUINO_DUE1.3V3; no longer B1.3.3V, Q13.G, Q14.G, Q2.G, Q3.G, R26.2, R28.2, R4.2, R6.2
- net 5V: now also ARDUINO_DUE1.5V, R4.2; no longer B1.5V@0, R25.2, R27.2, R5.2
- net D10: now also ARDUINO_DUE1.10; no longer B1.10
- net D11: now also ARDUINO_DUE1.11; no longer B1.11
- net D12: now also ARDUINO_DUE1.12; no longer B1.12
- net D13: now also ARDUINO_DUE1.13; no longer B1.13
- net D14: now also ARDUINO_DUE1.TX3_14; no longer B1.14(TX3)
- net D15: now also ARDUINO_DUE1.RX3_15; no longer B1.15(RX3)
- net D2: now also ARDUINO_DUE1.2; no longer B1.2
- net D22: now also ARDUINO_DUE1.22; no longer B1.22
- net D23: now also ARDUINO_DUE1.23; no longer B1.23
- net D24: now also ARDUINO_DUE1.24; no longer B1.24
- net D25: now also ARDUINO_DUE1.25; no longer B1.25
- net D26: now also ARDUINO_DUE1.26; no longer B1.26
- net D27: now also ARDUINO_DUE1.27; no longer B1.27
- net D28: now also ARDUINO_DUE1.28; no longer B1.28
- net D29: now also ARDUINO_DUE1.29; no longer B1.29
- net D3: now also ARDUINO_DUE1.3; no longer B1.3
- net D30: now also ARDUINO_DUE1.30; no longer B1.30
- net D31: now also ARDUINO_DUE1.31; no longer B1.31
- net D32: now also ARDUINO_DUE1.32; no longer B1.32
- net D33: now also ARDUINO_DUE1.33; no longer B1.33
- net D34: now also ARDUINO_DUE1.34; no longer B1.34
- net D35: now also ARDUINO_DUE1.35; no longer B1.35
- net D4: now also ARDUINO_DUE1.4; no longer B1.4
- net D5: now also ARDUINO_DUE1.5; no longer B1.5
- net D6: now also ARDUINO_DUE1.6; no longer B1.6
- net D7: now also ARDUINO_DUE1.7; no longer B1.7
- net D8: now also ARDUINO_DUE1.8; no longer B1.8
- net D9: now also ARDUINO_DUE1.9; no longer B1.9
- net GND: now also ARDUINO_DUE1.GND; no longer B1.GND@0, X1-2.S
- net RX: now also ARDUINO_DUE1.RX0<0; no longer B1.0(RX0), Q13.D, R25.1
- net SCL_OUT: now also ARDUINO_DUE1.SCL_21, R3.1; no longer Q3.D, R5.1
- net SDA_OUT: now also ARDUINO_DUE1.SDA_20, R4.1; no longer Q2.D, R3.1
- net TX: now also ARDUINO_DUE1.TX0>1; no longer B1.1(TX0), Q14.D, R27.1
Other:
- moved on the sheet: R3, R4

Commit message: Finished Layout for Relay support circuitry
Parts:
- removed 12V, GND: (no value), wirepad:3,81/1,4
- removed ENCODER_OUTPUT1: (no value), con-lstb:MA04-1
- removed R10, R11: 10K, rcl:R-US_R0603
- added C1, C2: (no value), adafruit:C-US050-045X075
- added IC1: 7805TV, linear:7805TV
- added LED1, LED2, LED3, LED4, LED5, LED6, LED7: (no value), led:LEDCHIP-LED0603
- added R5, R6: 25K, rcl:R-US_R0603
- added S1, S2, S3, S4, S5, S6, S7: (no value), switch-dil:DS01E
- added U$1: MEGA-FIT_RA_2, RSX:MEGA-FIT_RA_2
- R1, R2, R7, R8, R9: value 10K -> 25K
- renumbered JP10 to M-5, JP11 to M-6, JP14 to M-7, JP6 to M-1, JP7 to M-2, JP8 to M-3, JP9 to M-4
Connections:
- removed net 12V: 12V.P, ARDUINO_DUE1.VIN, M-1.7, M-1.8, M-2.7, M-2.8, M-3.7, M-3.8, M-4.7, M-4.8, M-5.7, M-5.8, M-6.7, M-6.8, M-7.7, M-7.8
- removed net 3.3V: ARDUINO_DUE1.3V3, MD_OUT_1.4, MD_OUT_2.4, MD_OUT_3.4, MD_OUT_4.4, MD_OUT_5.4, MD_OUT_6.4, MD_OUT_7.4, R1.2, R10.2, R11.2, R2.2, R7.2, R8.2, R9.2
- removed net RX: ARDUINO_DUE1.RX0<0
- removed net TX: ARDUINO_DUE1.TX0>1
- new net 3V3: ARDUINO_DUE1.3V3, S1.1, S2.1, S3.1, S4.1, S5.1, S6.1, S7.1
- new net D0: ARDUINO_DUE1.RX0<0, MD_OUT_7.2
- new net D1: ARDUINO_DUE1.TX0>1, MD_OUT_6.2
- new net N$1: LED1.A, R1.2
- new net N$28: LED3.A, R5.2
- new net N$3: LED2.A, R2.2
- new net N$30: LED4.A, R6.2
- new net N$32: LED5.A, R7.2
- new net N$34: LED6.A, R8.2
- new net N$36: LED7.A, R9.2
- new net N1: MD_OUT_2.4, R8.1, S6.2
- new net N2: MD_OUT_3.4, R7.1, S5.2
- new net N3: MD_OUT_4.4, R6.1, S4.2
- new net N4: MD_OUT_5.4, R5.1, S3.2
- new net N5: MD_OUT_6.4, R2.1, S2.2
- new net N6: MD_OUT_7.4, R1.1, S1.2
- new net N7: MD_OUT_1.4, R9.1, S7.2
- new net V+: C2.1, IC1.VI, M-1.7, M-1.8, M-2.7, M-2.8, M-3.7, M-3.8, M-4.7, M-4.8, M-5.7, M-5.8, M-6.7, M-6.8, M-7.7, M-7.8, U$1.P$1
- new net VIN: ARDUINO_DUE1.VIN, C1.1, IC1.VO
- net 5V: no longer ENCODER_OUTPUT1.4
- net D10: now also MD_OUT_2.2; no longer MD_OUT_4.2
- net D11: now also MD_OUT_2.3; no longer MD_OUT_5.2
- net D12: now also MD_OUT_1.2; no longer MD_OUT_6.2
- net D13: now also MD_OUT_1.3; no longer MD_OUT_7.2
- net D14: no longer MD_OUT_2.2
- net D15: no longer MD_OUT_1.2
- net D2: now also MD_OUT_7.3; no longer MD_OUT_1.3
- net D23: no longer MD_OUT_7.5, R1.1
- net D25: no longer MD_OUT_6.5, R2.1
- net D27: no longer MD_OUT_5.5, R7.1
- net D29: no longer MD_OUT_4.5, R8.1
- net D3: now also MD_OUT_6.3; no longer MD_OUT_2.3
- net D31: no longer MD_OUT_3.5, R9.1
- net D33: no longer MD_OUT_2.5, R10.1
- net D35: no longer MD_OUT_1.5, R11.1
- net D4: now also MD_OUT_5.2; no longer MD_OUT_3.3
- net D5: now also MD_OUT_5.3; no longer MD_OUT_4.3
- net D6: now also MD_OUT_4.2; no longer MD_OUT_5.3
- net D7: now also MD_OUT_4.3; no longer MD_OUT_6.3
- net D8: now also MD_OUT_3.2; no longer MD_OUT_7.3
- net D9: now also MD_OUT_3.3; no longer MD_OUT_3.2
- net GND: now also C1.2, C2.2, IC1.GND, LED1.C, LED2.C, LED3.C, LED4.C, LED5.C, LED6.C, LED7.C, U$1.P$2; no longer ENCODER_OUTPUT1.1, GND.P
- net SCL_OUT: no longer ENCODER_OUTPUT1.3
- net SDA_OUT: no longer ENCODER_OUTPUT1.2
Other:
- moved on the sheet: R1, R2, R7, R8, R9
